File: project_02/EAGLE/FitnessTracker.brd (EAGLE design)
At the start: 81.9 x 67 mm, 23 parts, among them SW1 PUSH_BUTTON, SW2 PUSH_BUTTON, SW3 PUSH_BUTTON

Commit message: Final touches to project 2
Routing:
- net GND: track 8.09 -> 1.10 mm
- net VDD_3P3V: track 8.06 -> 5.52 mm
Changed lines of the file:
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@@
 <layers>
 <layer number="1" name="Top" color="4" fill="1" visible="yes" active="yes"/>
-<layer number="2" name="Route2" color="16" fill="1" visible="no" active="yes"/>
+<layer number="2" name="Route2" color="16" fill="1" visible="yes" active="yes"/>
 <layer number="3" name="Route3" color="17" fill="1" visible="no" active="no"/>
 <layer number="4" name="Route4" color="18" fill="1" visible="no" active="no"/>
@@
 <layer number="13" name="Route13" color="21" fill="1" visible="no" active="no"/>
 <layer number="14" name="Route14" color="22" fill="1" visible="no" active="no"/>
-<layer number="15" name="Route15" color="23" fill="1" visible="no" active="yes"/>
+<layer number="15" name="Route15" color="23" fill="1" visible="yes" active="yes"/>
 <layer number="16" name="Bottom" color="1" fill="1" visible="yes" active="yes"/>
 <layer number="17" name="Pads" color="2" fill="1" visible="yes" active="yes"/>
@@
 <vertex x="-5.08" y="81.28"/>
 </polygon>
-<wire x1="68.58" y1="38.735" x2="68.58" y2="36.195" width="0.254" layer="2"/>
 </signal>
 <signal name="GND">
@@
 <wire x1="78.5749" y1="9.525" x2="77.47" y2="9.525" width="0.254" layer="1"/>
 <via x="77.47" y="9.525" extent="1-16" drill="0.3048" diameter="0.6096"/>
-<wire x1="15.24" y1="55.245" x2="19.05" y2="55.245" width="0.254" layer="2"/>
-<wire x1="68.58" y1="43.815" x2="68.58" y2="46.99" width="0.254" layer="15"/>
 </signal>
 <signal name="MODE_BUTTON">
